File: kicad/stm32f103_feather/stm32f103_feather.kicad_pcb (KiCad board)
At the start: 2 copper layers, 50.8 x 22.9 mm, 28 parts, among them J1 Conn_01x16, J2 Conn_01x12, J3 Conn_01x04, J4 USB_B_Micro, J5 HEADER-FEMALE-2POS-TH-1x02-JS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, SW1 SW_Push, U1 STM32F103CBTx, U2 AMS1117-3.3, Y1 8MHz

Commit message: daily updates
Parts:
- added C14: 10u, Capacitor_SMD:C_0603_1608Metric_Pad1.05x0.95mm_HandSolder, B.Cu at (141.9, 89.5)
- added D4: Yellow, Diode_SMD:D_0603_1608Metric_Pad1.05x0.95mm_HandSolder, B.Cu at (145.9, 91.1)
- added JP1: Boot-select, Connector_PinHeader_2.54mm:PinHeader_1x03_P2.54mm_Vertical, F.Cu at (172.7, 91.4)
- added R4: 10k, Resistor_SMD:R_0603_1608Metric_Pad1.05x0.95mm_HandSolder, B.Cu at (141.9, 91.2)
- added R5: 2k2, Resistor_SMD:R_0603_1608Metric_Pad1.05x0.95mm_HandSolder, B.Cu at (145.9, 89.5)
- added U3: MCP73831-2-OT, Package_TO_SOT_SMD:SOT-23-5, B.Cu at (137.6, 90.5)
- J1: value Conn_01x16 -> Bottom-conn
- J2: value Conn_01x12 -> Top-conn
- J3: value Conn_01x04 -> Debug-conn
- J5: value HEADER-FEMALE-2POS-TH-1x02-JST-PH -> JST-LiPo-conn; footprint Connector_JST:JST_GH_SM02B-GHS-TB_1x02-1MP_P1.25mm_Horizontal -> Connector_JST:JST_PH_S2B-PH-SM4-TB_1x02-1MP_P2.00mm_Horizontal; moved to B.Cu
- U2: moved to F.Cu
- moved C6 31.5 mm to (169.6, 80.6)
- moved C5 28.1 mm to (169.6, 82.0)
- moved C9 28.0 mm to (162.7, 80.6)
- moved C4 26.6 mm to (138.6, 90.8), turned to 0 degrees
- moved U2 25.3 mm to (138.8, 84.5), turned to 0 degrees
- moved C10 23.9 mm to (162.7, 82.0)
- moved C13 23.6 mm to (138.5, 89.2), turned to 180 degrees
- moved C8 21.4 mm to (168.5, 94.6), turned to 270 degrees
- moved C7 15.9 mm to (170.2, 94.6), turned to 270 degrees
- moved C2 6.77 mm to (154.1, 87.8), turned to 90 degrees
- moved C12 4.29 mm to (156.7, 91.6), turned to 180 degrees
- moved C11 4.06 mm to (156.7, 93.0)
- moved Y1 4.03 mm to (156.8, 86.1), turned to 270 degrees
- moved U1 3.80 mm to (164.2, 88.2)
- moved C1 3.58 mm to (154.1, 84.4), turned to 90 degrees
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Connections:
- C1 pad 2: /osc_out -> /osc_in
- C12 pad 1: GND -> /vref
- C12 pad 2: /vref -> GND
- C2 pad 1: /osc_in -> /osc_out
- C4 pad 1: /3vo -> GND
- C4 pad 2: GND -> /3vo
- J1 pad 1: /rst -> (no net)
- J2 pad 10: Net-(J2-Pad10) -> /nss
- J2 pad 2: /en -> (no net)
- J2 pad 4: Net-(J2-Pad4) -> /pb8
- J2 pad 5: Net-(J2-Pad5) -> /pb9
- J2 pad 6: Net-(J2-Pad6) -> /pb10
- J2 pad 7: Net-(J2-Pad7) -> /pb11
- J2 pad 8: Net-(J2-Pad8) -> /pa6
- J2 pad 9: Net-(J2-Pad9) -> /pa7
- J4 pad 4: Net-(J4-Pad4) -> (no net)
- R2 pad 2: Net-(R2-Pad2) -> /pa8
- U1 pad 1: Net-(U1-Pad1) -> (no net)
- U1 pad 10: Net-(U1-Pad10) -> /a0
- U1 pad 11: Net-(U1-Pad11) -> /a1
- U1 pad 12: Net-(U1-Pad12) -> /a2
- U1 pad 13: Net-(U1-Pad13) -> /a3
- U1 pad 14: Net-(U1-Pad14) -> /a4
- U1 pad 15: Net-(U1-Pad15) -> /a5
- U1 pad 16: Net-(U1-Pad16) -> /pa6
- U1 pad 17: Net-(U1-Pad17) -> /pa7
- U1 pad 18: Net-(U1-Pad18) -> (no net)
- U1 pad 19: Net-(U1-Pad19) -> (no net)
- U1 pad 2: Net-(U1-Pad2) -> (no net)
- U1 pad 20: Net-(U1-Pad20) -> (no net)
- U1 pad 21: /tx -> /pb10
- U1 pad 22: /rx -> /pb11
- U1 pad 25: Net-(U1-Pad25) -> /nss
- U1 pad 26: Net-(U1-Pad26) -> /sck
- U1 pad 27: Net-(U1-Pad27) -> /mi
- U1 pad 28: Net-(U1-Pad28) -> /mo
- U1 pad 29: Net-(U1-Pad29) -> /pa8
- U1 pad 30: Net-(U1-Pad30) -> /tx
- U1 pad 31: Net-(U1-Pad31) -> /rx
- U1 pad 38: Net-(U1-Pad38) -> (no net)
- U1 pad 39: Net-(U1-Pad39) -> (no net)
- U1 pad 40: Net-(U1-Pad40) -> (no net)
- U1 pad 41: Net-(U1-Pad41) -> (no net)
- U1 pad 44: Net-(U1-Pad44) -> /boot
- U1 pad 45: Net-(U1-Pad45) -> /pb8
- U1 pad 46: Net-(U1-Pad46) -> /pb9
- U1 pad 5: Net-(U1-Pad5) -> (no net)
- U1 pad 6: Net-(U1-Pad6) -> (no net)
- Y1 pad 1: /osc_out -> /osc_in
- Y1 pad 2: /osc_in -> /osc_out
Routing:
- net /gnd: vias 0 -> 4
- net (no net): vias 4 -> 0

Commit message: daily updates
Parts:
- moved R3 18.4 mm to (169.4, 90.3), turned to 270 degrees
- moved R2 18.2 mm to (167.9, 90.3), turned to 270 degrees
- moved D3 17.5 mm to (169.4, 86.5), turned to 90 degrees
- moved D2 17.4 mm to (167.9, 86.5), turned to 90 degrees
- moved C4 12.9 mm to (148.7, 82.8), turned to 180 degrees
- moved U2 2.56 mm to (141.4, 84.5)
- moved C12 2.54 mm to (154.2, 91.6)
- moved U1 2.54 mm to (161.7, 88.2)
- moved C1 2.54 mm to (151.5, 84.4)
- moved C10 2.54 mm to (160.2, 82.0)
- moved C11 2.54 mm to (154.2, 93.0)
- moved C2 2.54 mm to (151.5, 87.8)
- moved C5 2.54 mm to (167.0, 82.0)
- moved C6 2.54 mm to (167.0, 80.6)
- moved C9 2.54 mm to (160.2, 80.6)
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
Commit message: daily update
Parts:
- added Q1: SI2301CDS, Package_TO_SOT_SMD:SOT-23, F.Cu at (136.0, 83.6)
- added R6: 100k, Resistor_SMD:R_0603_1608Metric_Pad1.05x0.95mm_HandSolder, F.Cu at (136.8, 87.0)
- moved D3 33.5 mm to (136.8, 94.2), turned to 180 degrees
- moved R3 30.9 mm to (138.6, 92.6), turned to 0 degrees
- moved R2 17.5 mm to (152.5, 81.9), turned to 0 degrees
- moved D2 16.5 mm to (152.5, 80.4), turned to 180 degrees
- moved R4 10.2 mm to (149.1, 83.9)
- moved C14 10.2 mm to (149.1, 82.3)
- moved R5 10.2 mm to (153.1, 82.3)
- moved U3 10.2 mm to (144.8, 83.3)
- moved D4 10.2 mm to (153.2, 83.8)
- moved C13 8.88 mm to (147.1, 87.9)
- moved C9 4.53 mm to (156.3, 83.1), turned to 180 degrees
- moved C4 4.47 mm to (145.3, 79.9)
- moved D1 4.44 mm to (146.2, 84.6), turned to 90 degrees
- moved C10 3.86 mm to (156.3, 81.7), turned to 180 degrees
- moved R1 3.49 mm to (136.9, 95.6)
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Connections:
- C13 pad 2: /usb -> Net-(C13-Pad2)
- D1 pad 1: /usb -> Net-(C13-Pad2)
- D1 pad 2: /bat -> /usb
- J1 pad 1: (no net) -> /nrst
- J1 pad 4: /gnd -> GND
- J2 pad 4: /pb8 -> /cantx
- J2 pad 5: /pb9 -> /canrx
- J2 pad 6: /pb10 -> /pb5
- J2 pad 7: /pb11 -> /pb4
- J2 pad 8: /pa6 -> /pb3
- J2 pad 9: /pa7 -> /pa15
- J3 pad 2: /gnd -> GND
- R2 pad 2: /pa8 -> /LED
- U1 pad 16: /pa6 -> (no net)
- U1 pad 17: /pa7 -> (no net)
- U1 pad 21: /pb10 -> /tx
- U1 pad 22: /pb11 -> /rx
- U1 pad 29: /pa8 -> (no net)
- U1 pad 3: /osc_in -> (no net)
- U1 pad 30: /tx -> (no net)
- U1 pad 31: /rx -> (no net)
- U1 pad 38: (no net) -> /pa15
- U1 pad 39: (no net) -> /pb3
- U1 pad 4: /osc_out -> /LED
- U1 pad 40: (no net) -> /pb4
- U1 pad 41: (no net) -> /pb5
- U1 pad 45: /pb8 -> /canrx
- U1 pad 46: /pb9 -> /cantx
- U1 pad 5: (no net) -> /osc_in
- U1 pad 6: (no net) -> /osc_out
- U2 pad 3: /usb -> Net-(C13-Pad2)
Routing:
- net /usb_dm: track 0.00 -> 43.1 mm, vias 0 -> 2
- net /usb_dp: track 0.00 -> 40.9 mm, vias 0 -> 2
- net /3vo: track 0.00 -> 38.9 mm, vias 0 -> 2
- net GND: track 0.00 -> 34.6 mm, vias 0 -> 13
- net /nrst: track 0.00 -> 32.1 mm, vias 0 -> 3
- net /usb: track 0.00 -> 27.5 mm
- net /vref: track 0.00 -> 25.8 mm
- net /nss: track 0.00 -> 21.1 mm, vias 0 -> 2
- net /a0: track 0.00 -> 19.1 mm
- net /boot: track 0.00 -> 16.6 mm, vias 0 -> 1
- net /a1: track 0.00 -> 16.4 mm
- net /swclk: track 0.00 -> 15.5 mm, vias 0 -> 1
- net /sda: track 0.00 -> 15.3 mm, vias 0 -> 1
- net /mo: track 0.00 -> 14.7 mm
- net /sck: track 0.00 -> 14.6 mm
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- added copper zone on B.Cu, net GND
- added copper zone on F.Cu, net GND

Commit message: daily updates
Parts:
- added J6: vrtc, Resistor_SMD:R_0402_1005Metric, F.Cu at (155.6, 85.7)
- C11, C12: footprint Capacitor_SMD:C_0603_1608Metric_Pad1.05x0.95mm_HandSolder -> Capacitor_SMD:C_0805_2012Metric_Pad1.15x1.40mm_HandSolder; moved to B.Cu
- C14: footprint Capacitor_SMD:C_0603_1608Metric_Pad1.05x0.95mm_HandSolder -> Capacitor_SMD:C_0805_2012Metric_Pad1.15x1.40mm_HandSolder
- D4: footprint Diode_SMD:D_0603_1608Metric_Pad1.05x0.95mm_HandSolder -> Diode_SMD:D_0805_2012Metric_Pad1.15x1.40mm_HandSolder
- R4, R5: footprint Resistor_SMD:R_0603_1608Metric_Pad1.05x0.95mm_HandSolder -> Resistor_SMD:R_0805_2012Metric_Pad1.15x1.40mm_HandSolder
- moved C14 5.35 mm to (144.0, 83.9), turned to 90 degrees
- moved D4 2.75 mm to (150.9, 82.3), turned to 180 degrees
- moved U3 2.20 mm to (146.9, 83.9), turned to 0 degrees
- moved R4 1.98 mm to (150.9, 84.8)
- moved C11 1.81 mm to (154.1, 92.8), turned to 270 degrees
- moved C4 1.56 mm to (146.7, 80.7)
- moved C7 1.39 mm to (171.7, 95.2), turned to 180 degrees
- moved C12 1.37 mm to (156.1, 92.8)
- moved R5 1.37 mm to (154.1, 83.3), turned to 270 degrees
- moved D3 0.51 mm to (136.8, 93.7)
- moved JP1 0.51 mm to (172.2, 91.4)
- moved C3 0.51 mm to (138.6, 90.6)
- moved R1 0.51 mm to (136.9, 95.1)
- moved R3 0.51 mm to (138.6, 92.1)
- moved Q1 0.34 mm to (135.6, 83.4)
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Connections:
- J2 pad 2: (no net) -> /en
- J4 pad 4: (no net) -> Net-(J4-Pad4)
- U1 pad 1: (no net) -> /vrtc
- U1 pad 16: (no net) -> Net-(U1-Pad16)
- U1 pad 17: (no net) -> Net-(U1-Pad17)
- U1 pad 18: (no net) -> Net-(U1-Pad18)
- U1 pad 19: (no net) -> Net-(U1-Pad19)
- U1 pad 2: (no net) -> Net-(U1-Pad2)
- U1 pad 20: (no net) -> Net-(U1-Pad20)
- U1 pad 29: (no net) -> Net-(U1-Pad29)
- U1 pad 3: (no net) -> Net-(U1-Pad3)
- U1 pad 30: (no net) -> Net-(U1-Pad30)
- U1 pad 31: (no net) -> Net-(U1-Pad31)
Routing:
- net /3vo: track 38.9 -> 106.0 mm, vias 2 -> 6
- net GND: track 34.6 -> 95.1 mm, vias 13 -> 17
- net /bat: track 10.7 -> 25.2 mm
- net /usb: track 27.5 -> 42.1 mm
- net Net-(R5-Pad2): track 0.00 -> 8.88 mm
- net /vref: track 25.8 -> 33.2 mm, vias 0 -> 1
- net /nss: track 21.1 -> 26.0 mm
- net /vrtc: track 0.00 -> 2.23 mm
- net Net-(D4-Pad1): track 0.00 -> 2.14 mm
- net Net-(R4-Pad1): track 0.00 -> 1.94 mm
- net /LED: track 7.58 -> 8.60 mm
- net /nrst: track 32.1 -> 32.9 mm
Other:
- rule via_min_size: 0.4 -> 0.45
- board text added: "3V3"
- board text added: "A0"
- board text added: "A1"
- board text added: "A2"
- board text added: "A3"
- board text added: "A4"
- board text added: "A5"
- board text added: "BAT"
- board text added: "GND"
- board text added: "MISO"
- board text added: "MOSI"
- board text added: "NC"
- board text added: "NRST"
- board text added: "PA15"
- board text added: "PB12"
- board text added: "PB3"
- board text added: "PB4"
- board text added: "PB5"
- board text added: "PB8"
- board text added: "PB9"
- board text added: "RX"
- board text added: "SCK"
- board text added: "SCL"
- board text added: "SDA"
- board text added: "TX"
- board text added: "USB"
- board text added: "VREF"
- board text added: "stm32f103cb feather-compatible ipyd-2020"

Commit message: daily updates
Parts:
- removed J6: vrtc, Resistor_SMD:R_0402_1005Metric
- added R7: 100k, Resistor_SMD:R_0805_2012Metric_Pad1.15x1.40mm_HandSolder, B.Cu at (146.3, 90.9)
- added R8: 100k, Resistor_SMD:R_0805_2012Metric_Pad1.15x1.40mm_HandSolder, B.Cu at (144.1, 90.9)
- added usart1: Conn_01x03, Jumper:SolderJumper-3_P1.3mm_Open_Pad1.0x1.5mm, B.Cu at (161.5, 92.2)
- added vrtc1: vrtc, Resistor_SMD:R_0402_1005Metric, F.Cu at (155.6, 85.7)
Connections:
- J2 pad 2: /en -> (no net)
- J4 pad 4: Net-(J4-Pad4) -> (no net)
- U1 pad 16: Net-(U1-Pad16) -> /batvtest
- U1 pad 17: Net-(U1-Pad17) -> (no net)
- U1 pad 18: Net-(U1-Pad18) -> (no net)
- U1 pad 19: Net-(U1-Pad19) -> (no net)
- U1 pad 2: Net-(U1-Pad2) -> (no net)
- U1 pad 20: Net-(U1-Pad20) -> (no net)
- U1 pad 3: Net-(U1-Pad3) -> (no net)
Routing:
- net /bat: track 25.2 -> 51.6 mm
- net /batvtest: track 0.00 -> 21.5 mm, vias 0 -> 1
- net Net-(U1-Pad31): track 0.00 -> 8.20 mm, vias 0 -> 1
- net Net-(U1-Pad30): track 0.00 -> 6.86 mm, vias 0 -> 1
- net Net-(U1-Pad29): track 0.00 -> 5.75 mm, vias 0 -> 1
- net GND: track 95.1 -> 96.6 mm

Commit message: daily updates
Parts:
- added J6: Conn_01x04, Connector_PinHeader_1.00mm:PinHeader_1x04_P1.00mm_Vertical_SMD_Pin1Left, B.Cu at (129.4, 87.6)
Connections:
- J2 pad 2: (no net) -> /en
- J4 pad 4: (no net) -> Net-(J4-Pad4)
- U1 pad 17: (no net) -> Net-(U1-Pad17)
- U1 pad 18: (no net) -> Net-(U1-Pad18)
- U1 pad 19: (no net) -> Net-(U1-Pad19)
- U1 pad 2: (no net) -> Net-(U1-Pad2)
- U1 pad 20: (no net) -> Net-(U1-Pad20)
- U1 pad 3: (no net) -> Net-(U1-Pad3)
Routing:
- net GND: track 96.6 -> 100.5 mm, vias 17 -> 18
- net /usb_dm: track 43.1 -> 47.0 mm, vias 2 -> 3
- net /usb_dp: track 40.9 -> 43.1 mm, vias 2 -> 3
- net /usb: track 42.1 -> 44.0 mm, vias 0 -> 1
Other:
- board text added: "0"
- board text added: "1"
- board text added: "BOOT"
- board text added: "SWCLK"
- board text added: "SWDIO"
- board text added: "USB_DM"
- board text added: "USB_DP"
- board text added: "VUSB"
