File: kicad/stm32f103_feather/stm32f103_feather.sch (KiCad schematic (older format))
At the start: 28 parts, among them J1 Conn_01x16, J2 Conn_01x12, J3 Conn_01x04, J4 USB_B_Micro, J5 HEADER-FEMALE-2POS-TH-1x02-JS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, SW1 SW_Push, U1 STM32F103CBTx, U2 AMS1117-3.3, Y1 8MHz

Commit message: daily updates
Parts:
- removed J5: HEADER-FEMALE-2POS-TH-1x02-JST-PH, Connector_JST:JST_GH_SM02B-GHS-TB_1x02-1MP_P1.25mm_Horizontal, symbol wickerlib:HEADER-FEMALE-2POS-TH-1x02-JST-PH
- added C14: 10u, Capacitor_SMD:C_0603_1608Metric_Pad1.05x0.95mm_HandSolder, symbol Device:C_Small
- added D4: Yellow, Diode_SMD:D_0603_1608Metric_Pad1.05x0.95mm_HandSolder, symbol Device:LED_Small
- added J5: JST-LiPo-conn, Connector_JST:JST_PH_S2B-PH-SM4-TB_1x02-1MP_P2.00mm_Horizontal, symbol Connector_Generic:Conn_01x02
- added JP1: Boot-select, Connector_PinHeader_2.54mm:PinHeader_1x03_P2.54mm_Vertical, symbol Jumper:SolderJumper_3_Open
- added R4: 10k, Resistor_SMD:R_0603_1608Metric_Pad1.05x0.95mm_HandSolder, symbol Device:R_Small
- added R5: 2k2, Resistor_SMD:R_0603_1608Metric_Pad1.05x0.95mm_HandSolder, symbol Device:R_Small
- added U3: MCP73831-2-OT, Package_TO_SOT_SMD:SOT-23-5, symbol Battery_Management:MCP73831-2-OT
- J1: value Conn_01x16 -> Bottom-conn
- J2: value Conn_01x12 -> Top-conn
- J3: value Conn_01x04 -> Debug-conn
Connections:
- net labels added: boot, nss, pa6, pa7, pa8, pb10, pb11, pb8, pb9
- wire segments 55 -> 70
- no-connect marks 1 -> 0
Other:
- note added: "Place on bottom"
- moved on the sheet: C1, C13, C2, C3, C4, D1, D2, D3, J1, J2, J3, J4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

Commit message: daily update
Parts:
- added Q1: SI2301CDS, Package_TO_SOT_SMD:SOT-23, symbol Transistor_FET:Si2371EDS
- added R6: 100k, Resistor_SMD:R_0603_1608Metric_Pad1.05x0.95mm_HandSolder, symbol Device:R_Small
Connections:
- net gnd is gone; now on net GND: J1.4 (Pin_4), J3.2 (Pin_2)
- net rst is gone; now on net nrst: J1.1 (Pin_1)
- net GND: now also R6.2
- net bat: now also Q1.3 (D); no longer D1.2 (A)
- net osc_in: now also U1.5 (PD0); no longer U1.3 (PC14)
- net osc_out: now also U1.6 (PD1); no longer U1.4 (PC15)
- net rx: now also U1.22 (PB11); no longer U1.31 (PA10)
- net tx: now also U1.21 (PB10); no longer U1.30 (PA9)
- net usb: now also D1.2 (A), Q1.1 (G), R6.1; no longer C13.2, D1.1 (K), U2.3 (VI)
- net pa15: now reaches U1.38 (PA15)
- net pa15: now also J2.9 (Pin_9)
- net pb3: now reaches U1.39 (PB3)
- net pb3: now also J2.8 (Pin_8)
- net pb4: now reaches U1.40 (PB4)
- net pb4: now also J2.7 (Pin_7)
- net pb5: now reaches U1.41 (PB5)
- net pb5: now also J2.6 (Pin_6)
- net pa6: no longer names the net of U1.16 (PA6)
- net pa6: no longer J2.8 (Pin_8)
- net pa7: no longer names the net of U1.17 (PA7)
- net pa7: no longer J2.9 (Pin_9)
- net pa8: no longer names the net of U1.29 (PA8)
- net pa8: no longer R2.2
- removed net pb10: J2.6 (Pin_6), U1.21 (PB10)
- removed net pb11: J2.7 (Pin_7), U1.22 (PB11)
- net pb8 renamed canrx
- net canrx: now also J2.5 (Pin_5); no longer J2.4 (Pin_4)
- net pb9 renamed cantx
- net cantx: now also J2.4 (Pin_4); no longer J2.5 (Pin_5)
- new net: C13.2, D1.1 (K), Q1.2 (S), U2.3 (VI)
- new net LED: R2.2, U1.4 (PC15)
Other:
- moved on the sheet: C13, C4, D1, U2
Changed lines of the file:
@@
 usb
 Text Label 1300 950  0    50   ~ 0
-rst
+nrst
 Text Label 1300 1050 0    50   ~ 0
 3vo
@@
 sck
 $Comp
-L MCU_ST_STM32F1:STM32F103CBTx U1
-U 1 1 5F3A98EE
-P 9450 2900
-F 0 "U1" H 9750 1450 50  0000 C CNN
-F 1 "STM32F103CBTx" H 10000 1350 50  0000 C CNN
-F 2 "Package_QFP:LQFP-48_7x7mm_P0.5mm" H 8850 1500 50  0001 R CNN
-F 3 "http://www.st.com/st-web-ui/static/active/en/resource/technical/document/datasheet/CD00161566.pdf" H 9450 2900 50  0001 C CNN
-F 4 "C8304" H 9450 2900 50  0001 C CNN "LSCS"
-	1    9450 2900
-	1    0    0    -1
-$EndComp
-$Comp
 L Device:Crystal Y1
 U 1 1 5F397667
@@
 Text Label 7400 5500 0    50   ~ 0
 osc_out
-Text Label 8750 2400 2    50   ~ 0
+Text Label 8750 2000 2    50   ~ 0
 osc_in
-Text Label 8750 2500 2    50   ~ 0
+Text Label 8750 2100 2    50   ~ 0
 osc_out
 Text Label 8750 3300 2    50   ~ 0
@@
 Text Label 8750 3400 2    50   ~ 0
 sda
-Text Label 10050 3600 0    50   ~ 0
+Text Label 8750 3700 2    50   ~ 0
 tx
-Text Label 10050 3700 0    50   ~ 0
+Text Label 8750 3800 2    50   ~ 0
 rx
 $Comp
@@
 L Regulator_Linear:AMS1117-3.3 U2
 U 1 1 5F3A741F
-P 3800 4150
-F 0 "U2" H 3800 4392 50  0000 C CNN
-F 1 "AMS1117-3.3" H 3800 4301 50  0000 C CNN
-F 2 "Package_TO_SOT_SMD:SOT-223-3_TabPin2" H 3800 4350 50  0001 C CNN
-F 3 "http://www.advanced-monolithic.com/pdf/ds1117.pdf" H 3900 3900 50  0001 C CNN
-F 4 "C6186" H 3800 4150 50  0001 C CNN "LCSC"
-	1    3800 4150
+P 4200 4100
+F 0 "U2" H 4200 4342 50  0000 C CNN
+F 1 "AMS1117-3.3" H 4200 4251 50  0000 C CNN
+F 2 "Package_TO_SOT_SMD:SOT-223-3_TabPin2" H 4200 4300 50  0001 C CNN
+F 3 "http://www.advanced-monolithic.com/pdf/ds1117.pdf" H 4300 3850 50  0001 C CNN
+F 4 "C6186" H 4200 4100 50  0001 C CNN "LCSC"
+	1    4200 4100
 	1    0    0    -1
 $EndComp
@@
 L Device:C_Small C4
 U 1 1 5F3A8CEF
-P 4200 4300
-F 0 "C4" H 4292 4346 50  0000 L CNN
-F 1 "22u" H 4292 4255 50  0000 L CNN
-F 2 "Capacitor_SMD:C_0603_1608Metric_Pad1.05x0.95mm_HandSolder" H 4200 4300 50  0001 C CNN
-F 3 "~" H 4200 4300 50  0001 C CNN
-F 4 "C59461" H 4200 4300 50  0001 C CNN "LCSC"
-	1    4200 4300
-	1    0    0    1
-$EndComp
-Wire Wire Line
-	4200 4200 4200 4150
-Wire Wire Line
-	4200 4150 4100 4150
-Wire Wire Line
-	4200 4400 4200 4450
-Wire Wire Line
-	4200 4450 3800 4450
+P 4600 4250
+F 0 "C4" H 4692 4296 50  0000 L CNN
+F 1 "22u" H 4692 4205 50  0000 L CNN
+F 2 "Capacitor_SMD:C_0603_1608Metric_Pad1.05x0.95mm_HandSolder" H 4600 4250 50  0001 C CNN
+F 3 "~" H 4600 4250 50  0001 C CNN
+F 4 "C59461" H 4600 4250 50  0001 C CNN "LCSC"
+	1    4600 4250
+	1    0    0    1
+$EndComp
+Wire Wire Line
+	4600 4150 4600 4100
+Wire Wire Line
+	4600 4100 4500 4100
+Wire Wire Line
+	4600 4350 4600 4400
+Wire Wire Line
+	4600 4400 4200 4400
 $Comp
 L power:GND #PWR0103
 U 1 1 5F3A9B16
-P 3800 4450
-F 0 "#PWR0103" H 3800 4200 50  0001 C CNN
-F 1 "GND" H 3805 4277 50  0000 C CNN
-F 2 "" H 3800 4450 50  0001 C CNN
-F 3 "" H 3800 4450 50  0001 C CNN
-	1    3800 4450
-	1    0    0    -1
-$EndComp
-Connection ~ 3800 4450
+P 4200 4400
+F 0 "#PWR0103" H 4200 4150 50  0001 C CNN
+F 1 "GND" H 4205 4227 50  0000 C CNN
+F 2 "" H 4200 4400 50  0001 C CNN
+F 3 "" H 4200 4400 50  0001 C CNN
+	1    4200 4400
+	1    0    0    -1
+$EndComp
+Connection ~ 4200 4400
 $Comp
 L Device:C_Small C11
@@
 	9750 800  9850 800
 Wire Wire Line
-	9550 1400 9450 1400
-Wire Wire Line
-	9450 1400 9350 1400
-Connection ~ 9450 1400
-Wire Wire Line
 	9350 1400 9350 1000
-Connection ~ 9350 1400
 Connection ~ 9350 1000
 Wire Wire Line
@@
 $EndComp
 Wire Wire Line
-	9250 4400 9350 4400
-Wire Wire Line
-	9350 4400 9450 4400
-Connection ~ 9350 4400
-Wire Wire Line
 	9450 4400 9550 4400
 Connection ~ 9450 4400
@@
 	1    0    0    -1
 $EndComp
-Text Label 4200 4150 0    50   ~ 0
+Text Label 4600 4100 0    50   ~ 0
 3vo
 $Comp
 L Device:D_Schottky_Small D1
 U 1 1 5F3C984B
-P 3050 3900
-F 0 "D1" H 3050 3695 50  0000 C CNN
-F 1 "B5819W" H 3050 3786 50  0000 C CNN
-F 2 "Diode_SMD:D_SOD-123" V 3050 3900 50  0001 C CNN
-F 3 "~" V 3050 3900 50  0001 C CNN
-F 4 "C8598" H 3050 3900 50  0001 C CNN "LCSC"
-	1    3050 3900
+P 3100 4100
+F 0 "D1" H 3100 3895 50  0000 C CNN
+F 1 "B5819W" H 3100 3986 50  0000 C CNN
+F 2 "Diode_SMD:D_SOD-123" V 3100 4100 50  0001 C CNN
+F 3 "~" V 3100 4100 50  0001 C CNN
+F 4 "C8598" H 3100 4100 50  0001 C CNN "LCSC"
+	1    3100 4100
 	-1   0    0    1
 $EndComp
 Wire Wire Line
-	3150 3900 3350 3900
-Wire Wire Line
-	3350 3900 3350 4150
-Wire Wire Line
-	3350 4150 3500 4150
-Connection ~ 3350 4150
-Wire Wire Line
-	2800 3900 2950 3900
-Wire Wire Line
-	2800 4150 3350 4150
-Text Label 2800 4150 2    50   ~ 0
+	3750 3850 3750 4100
+Wire Wire Line
+	3750 4100 3900 4100
+Connection ~ 3750 4100
+Wire Wire Line
+	3200 4100 3750 4100
+Text Label 2750 3300 2    50   ~ 0
 usb
-Text Label 2800 3900 2    50   ~ 0
+Text Label 3750 3300 2    50   ~ 0
 bat
 $Comp
 L Device:C_Small C13
 U 1 1 5F3CE620
-P 3350 4300
-F 0 "C13" H 3258 4254 50  0000 R CNN
-F 1 "10u" H 3258 4345 50  0000 R CNN
-F 2 "Capacitor_SMD:C_0603_1608Metric_Pad1.05x0.95mm_HandSolder" H 3350 4300 50  0001 C CNN
-F 3 "~" H 3350 4300 50  0001 C CNN
-F 4 "C19702" H 3350 4300 50  0001 C CNN "LCSC"
-	1    3350 4300
-	1    0    0    1
-$EndComp
-Wire Wire Line
-	3350 4200 3350 4150
-Wire Wire Line
-	3350 4400 3350 4450
-Wire Wire Line
-	3350 4450 3800 4450
+P 3750 4250
+F 0 "C13" H 3658 4204 50  0000 R CNN
+F 1 "10u" H 3658 4295 50  0000 R CNN
+F 2 "Capacitor_SMD:C_0603_1608Metric_Pad1.05x0.95mm_HandSolder" H 3750 4250 50  0001 C CNN
+F 3 "~" H 3750 4250 50  0001 C CNN
+F 4 "C19702" H 3750 4250 50  0001 C CNN "LCSC"
+	1    3750 4250
+	1    0    0    1
+$EndComp
+Wire Wire Line
+	3750 4150 3750 4100
+Wire Wire Line
+	3750 4350 3750 4400
+Wire Wire Line
+	3750 4400 4200 4400
 $Comp
 L Device:LED_Small D2
@@
 Text Label 1300 1650 0    50   ~ 0
 a3
-Text Label 1300 1750 0    50   ~ 0
-a4
-Text Label 1300 1850 0    50   ~ 0
-a5
 $Comp
 L power:GND #PWR0108
@@
 Text Label 10050 3000 0    50   ~ 0
 a3
-Text Label 10050 3100 0    50   ~ 0
-a4
-Text Label 10050 3200 0    50   ~ 0
-a5
 $Comp
 L Jumper:SolderJumper_3_Open JP1
@@
 Text Label 2100 2250 2    50   ~ 0
 nss
-Text Label 8750 3700 2    50   ~ 0
-pb10
-Text Label 8750 3800 2    50   ~ 0
-pb11
+Text Label 8750 3600 2    50   ~ 0
+cantx
+Text Label 2100 1650 2    50   ~ 0
+cantx
+Text Label 8750 2500 2    50   ~ 0
+LED
+Text Label 6400 6000 2    50   ~ 0
+LED
+$Comp
+L Transistor_FET:Si2371EDS Q1
+U 1 1 5F3B89AB
+P 3650 3650
+F 0 "Q1" H 3854 3696 50  0000 L CNN
+F 1 "SI2301CDS" H 3854 3605 50  0000 L CNN
+F 2 "Package_TO_SOT_SMD:SOT-23" H 3850 3575 50  0001 L CIN
+F 3 "http://www.vishay.com/docs/63924/si2371eds.pdf" H 3650 3650 50  0001 L CNN
+F 4 "C10487" H 3650 3650 50  0001 C CNN "LCSC"
+	1    3650 3650
+	1    0    0    -1
+$EndComp
+Wire Wire Line
+	3750 3300 3750 3450
+$Comp
+L Device:R_Small R6
+U 1 1 5F3C3394
+P 2750 4250
+F 0 "R6" H 2809 4296 50  0000 L CNN
+F 1 "100k" H 2809 4205 50  0000 L CNN
+F 2 "Resistor_SMD:R_0603_1608Metric_Pad1.05x0.95mm_HandSolder" H 2750 4250 50  0001 C CNN
+F 3 "~" H 2750 4250 50  0001 C CNN
+F 4 "C25803" H 2750 4250 50  0001 C CNN "LCSC"
+	1    2750 4250
+	1    0    0    -1
+$EndComp
+Wire Wire Line
+	3000 4100 2750 4100
+Wire Wire Line
+	2750 4100 2750 4150
+Wire Wire Line
+	2750 4350 2750 4400
+Wire Wire Line
+	2750 4400 3750 4400
+Connection ~ 3750 4400
+Wire Wire Line
+	3450 3650 2750 3650
+Wire Wire Line
+	2750 3650 2750 4100
+Connection ~ 2750 4100
+Wire Wire Line
+	2750 3300 2750 3650
+Connection ~ 2750 3650
+Text Label 3250 4400 0    50   ~ 0
+gnd
+Text Label 10050 3100 0    50   ~ 0
+a4
+Text Label 10050 3200 0    50   ~ 0
+a5
+Text Label 1300 1750 0    50   ~ 0
+a4
+Text Label 1300 1850 0    50   ~ 0
+a5
+Text Label 2100 1750 2    50   ~ 0
+canrx
 Text Label 8750 3500 2    50   ~ 0
-pb8
-Text Label 8750 3600 2    50   ~ 0
-pb9
-Text Label 2100 1650 2    50   ~ 0
-pb8
-Text Label 2100 1750 2    50   ~ 0
-pb9
+canrx
+Text Label 8750 3200 2    50   ~ 0
+pb5
+Text Label 8750 3100 2    50   ~ 0
+pb4
+Text Label 8750 3000 2    50   ~ 0
+pb3
+Connection ~ 9350 4400
+Wire Wire Line
+	9350 4400 9450 4400
+Wire Wire Line
+	9250 4400 9350 4400
+Connection ~ 9350 1400
+Connection ~ 9450 1400
+Wire Wire Line
+	9450 1400 9350 1400
+Wire Wire Line
+	9550 1400 9450 1400
+$Comp
+L MCU_ST_STM32F1:STM32F103CBTx U1
+U 1 1 5F3A98EE
+P 9450 2900
+F 0 "U1" H 9750 1450 50  0000 C CNN
+F 1 "STM32F103CBTx" H 10000 1350 50  0000 C CNN
+F 2 "Package_QFP:LQFP-48_7x7mm_P0.5mm" H 8850 1500 50  0001 R CNN
+F 3 "http://www.st.com/st-web-ui/static/active/en/resource/technical/document/datasheet/CD00161566.pdf" H 9450 2900 50  0001 C CNN
+F 4 "C8304" H 9450 2900 50  0001 C CNN "LSCS"
+	1    9450 2900
+	1    0    0    -1
+$EndComp
+Text Label 10050 4200 0    50   ~ 0
+pa15
+Text Label 2100 2150 2    50   ~ 0
+pa15
 Text Label 2100 1850 2    50   ~ 0
-pb10
+pb5
+Text Label 2100 2050 2    50   ~ 0
+pb3
 Text Label 2100 1950 2    50   ~ 0
-pb11
-Text Label 2100 2050 2    50   ~ 0
-pa6
-Text Label 2100 2150 2    50   ~ 0
-pa7
-Text Label 10050 3300 0    50   ~ 0
-pa6
-Text Label 10050 3400 0    50   ~ 0
-pa7
-Text Label 10050 3500 0    50   ~ 0
-pa8
-Text Label 6400 6000 2    50   ~ 0
-pa8
+pb4
 $EndSCHEMATC

Commit message: daily updates
Parts:
- added J6: vrtc, Resistor_SMD:R_0402_1005Metric, symbol Connector_Generic:Conn_01x02
- C11, C12, C14: footprint Capacitor_SMD:C_0603_1608Metric_Pad1.05x0.95mm_HandSolder -> Capacitor_SMD:C_0805_2012Metric_Pad1.15x1.40mm_HandSolder
- D4: footprint Diode_SMD:D_0603_1608Metric_Pad1.05x0.95mm_HandSolder -> Diode_SMD:D_0805_2012Metric_Pad1.15x1.40mm_HandSolder
- R4, R5: footprint Resistor_SMD:R_0603_1608Metric_Pad1.05x0.95mm_HandSolder -> Resistor_SMD:R_0805_2012Metric_Pad1.15x1.40mm_HandSolder
Connections:
- net GND: now also J6.1 (Pin_1)
- net vrtc: now reaches U1.1 (VBAT)
- net vrtc: now also J6.2 (Pin_2)
- no-connect marks 0 -> 12
Other:
- note added: "LiPo charger\n(Place on bottom)"
- note added: "Power supply"
- note removed: "Place on bottom"
- moved on the sheet: C1, C10, C11, C12, C13, C14, C2, C3, C4, C5, C6, C7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

Commit message: daily updates
Parts:
- added R7, R8: 100k, Resistor_SMD:R_0805_2012Metric_Pad1.15x1.40mm_HandSolder, symbol Device:R_Small
- added usart1: Conn_01x03, Jumper:SolderJumper-3_P1.3mm_Open_Pad1.0x1.5mm, symbol Connector_Generic:Conn_01x03
- renumbered J6 to vrtc1
Connections:
- net GND: now also R8.2
- net bat: now also R7.1
- net batvtest: now reaches U1.16 (PA6)
- net batvtest: now also R7.2, R8.1
- net at U1.29 (PA8): now also usart1.3 (Pin_3)
- net at U1.30 (PA9): now also usart1.2 (Pin_2)
- net at U1.31 (PA10): now also usart1.1 (Pin_1)
- no-connect marks 12 -> 8
Other:
- moved on the sheet: J5
Changed lines of the file:
@@
 Text Label 2550 3550 0    50   ~ 0
-usb_dm
-Text Label 9350 5450 0    50   ~ 0
 usb_dm
 $Comp
@@
 L power:GND #PWR0110
 U 1 1 5F3F0470
-P 5100 5550
-F 0 "#PWR0110" H 5100 5300 50  0001 C CNN
-F 1 "GND" H 5105 5377 50  0000 C CNN
-F 2 "" H 5100 5550 50  0001 C CNN
-F 3 "" H 5100 5550 50  0001 C CNN
-	1    5100 5550
-	1    0    0    -1
-$EndComp
-Text Label 5100 5450 0    50   ~ 0
+P 4900 5050
+F 0 "#PWR0110" H 4900 4800 50  0001 C CNN
+F 1 "GND" H 4905 4877 50  0000 C CNN
+F 2 "" H 4900 5050 50  0001 C CNN
+F 3 "" H 4900 5050 50  0001 C CNN
+	1    4900 5050
+	1    0    0    -1
+$EndComp
+Text Label 4900 4950 0    50   ~ 0
 bat
 $Comp
 L Connector_Generic:Conn_01x02 J5
 U 1 1 5F3A21F3
-P 4900 5550
-F 0 "J5" H 4818 5225 50  0000 C CNN
-F 1 "JST-LiPo-conn" H 4818 5316 50  0000 C CNN
-F 2 "Connector_JST:JST_PH_S2B-PH-SM4-TB_1x02-1MP_P2.00mm_Horizontal" H 4900 5550 50  0001 C CNN
-F 3 "~" H 4900 5550 50  0001 C CNN
-	1    4900 5550
+P 4700 5050
+F 0 "J5" H 4618 4725 50  0000 C CNN
+F 1 "JST-LiPo-conn" H 4618 4816 50  0000 C CNN
+F 2 "Connector_JST:JST_PH_S2B-PH-SM4-TB_1x02-1MP_P2.00mm_Horizontal" H 4700 5050 50  0001 C CNN
+F 3 "~" H 4700 5050 50  0001 C CNN
+	1    4700 5050
 	-1   0    0    1
 $EndComp
@@
 Wire Wire Line
 	8850 3050 8750 3050
-$Comp
-L MCU_ST_STM32F1:STM32F103CBTx U1
-U 1 1 5F3A98EE
-P 8750 4550
-F 0 "U1" H 9050 3100 50  0000 C CNN
-F 1 "STM32F103CBTx" H 9300 3000 50  0000 C CNN
-F 2 "Package_QFP:LQFP-48_7x7mm_P0.5mm" H 8150 3150 50  0001 R CNN
-F 3 "http://www.st.com/st-web-ui/static/active/en/resource/technical/document/datasheet/CD00161566.pdf" H 8750 4550 50  0001 C CNN
-F 4 "C8304" H 8750 4550 50  0001 C CNN "LSCS"
-	1    8750 4550
-	1    0    0    -1
-$EndComp
 Text Label 9350 5850 0    50   ~ 0
 pa15
@@
 Power supply
 Wire Notes Line
-	9750 6350 9750 2150
-Wire Notes Line
-	9750 2150 5550 2150
+	10300 6350 10300 2150
 Wire Notes Line
 	5550 2150 5550 6350
 Wire Notes Line
-	5550 6350 9750 6350
-Wire Notes Line
 	1200 2850 2850 2850
 Wire Notes Line
@@
 Wire Wire Line
 	3700 1700 3800 1700
-NoConn ~ 9350 5350
-NoConn ~ 9350 5250
-NoConn ~ 9350 5150
 NoConn ~ 9350 5050
-NoConn ~ 9350 4950
 NoConn ~ 8050 4550
 NoConn ~ 8050 4450
@@
 vrtc
 $Comp
-L Connector_Generic:Conn_01x02 J6
+L Connector_Generic:Conn_01x02 vrtc1
 U 1 1 5F4EC4D8
 P 8050 2950
-F 0 "J6" H 7968 2625 50  0000 C CNN
-F 1 "vrtc" H 7968 2716 50  0000 C CNN
+F 0 "vrtc1" H 8050 2750 50  0000 C CNN
+F 1 "vrtc" H 7968 2716 50  0001 C CNN
 F 2 "Resistor_SMD:R_0402_1005Metric" H 8050 2950 50  0001 C CNN
 F 3 "~" H 8050 2950 50  0001 C CNN
@@
 NoConn ~ 2550 3650
 NoConn ~ 2400 1600
+$Comp
+L Device:R_Small R7
+U 1 1 5F3D06A1
+P 4900 5600
+F 0 "R7" H 4959 5646 50  0000 L CNN
+F 1 "100k" H 4959 5555 50  0000 L CNN
+F 2 "Resistor_SMD:R_0805_2012Metric_Pad1.15x1.40mm_HandSolder" H 4900 5600 50  0001 C CNN
+F 3 "~" H 4900 5600 50  0001 C CNN
+F 4 "C25804" H 4900 5600 50  0001 C CNN "LCSC"
+	1    4900 5600
+	-1   0    0    -1
+$EndComp
+$Comp
+L Device:R_Small R8
+U 1 1 5F3D0C34
+P 4900 5900
+F 0 "R8" H 4959 5946 50  0000 L CNN
+F 1 "100k" H 4959 5855 50  0000 L CNN
+F 2 "Resistor_SMD:R_0805_2012Metric_Pad1.15x1.40mm_HandSolder" H 4900 5900 50  0001 C CNN
+F 3 "~" H 4900 5900 50  0001 C CNN
+F 4 "C25804" H 4900 5900 50  0001 C CNN "LCSC"
+	1    4900 5900
+	-1   0    0    -1
+$EndComp
+$Comp
+L power:GND #PWR0114
+U 1 1 5F3D132A
+P 4900 6100
+F 0 "#PWR0114" H 4900 5850 50  0001 C CNN
+F 1 "GND" H 4905 5927 50  0000 C CNN
+F 2 "" H 4900 6100 50  0001 C CNN
+F 3 "" H 4900 6100 50  0001 C CNN
+	1    4900 6100
+	1    0    0    -1
+$EndComp
+Wire Wire Line
+	4900 5500 4900 5400
+Wire Wire Line
+	4900 5400 4250 5400
+Connection ~ 4250 5400
+Wire Wire Line
+	4900 6000 4900 6100
+Text Label 5000 5750 0    50   ~ 0
+batvtest
+Wire Wire Line
+	4900 5700 4900 5750
+Wire Wire Line
+	5000 5750 4900 5750
+Connection ~ 4900 5750
+Wire Wire Line
+	4900 5750 4900 5800
+Text Label 9350 4950 0    50   ~ 0
+batvtest
+$Comp
+L Connector_Generic:Conn_01x03 usart1
+U 1 1 5F3DF3AE
+P 10100 5250
+F 0 "usart1" H 10100 5000 50  0000 C CNN
+F 1 "Conn_01x03" H 10018 5016 50  0001 C CNN
+F 2 "Jumper:SolderJumper-3_P1.3mm_Open_Pad1.0x1.5mm" H 10100 5250 50  0001 C CNN
+F 3 "~" H 10100 5250 50  0001 C CNN
+	1    10100 5250
+	1    0    0    1
+$EndComp
+Text Label 9350 5450 0    50   ~ 0
+usb_dm
+$Comp
+L MCU_ST_STM32F1:STM32F103CBTx U1
+U 1 1 5F3A98EE
+P 8750 4550
+F 0 "U1" H 9050 3100 50  0000 C CNN
+F 1 "STM32F103CBTx" H 9300 3000 50  0000 C CNN
+F 2 "Package_QFP:LQFP-48_7x7mm_P0.5mm" H 8150 3150 50  0001 R CNN
+F 3 "http://www.st.com/st-web-ui/static/active/en/resource/technical/document/datasheet/CD00161566.pdf" H 8750 4550 50  0001 C CNN
+F 4 "C8304" H 8750 4550 50  0001 C CNN "LSCS"
+	1    8750 4550
+	1    0    0    -1
+$EndComp
+Wire Wire Line
+	9350 5150 9900 5150
+Wire Wire Line
+	9900 5250 9350 5250
+Wire Wire Line
+	9350 5350 9900 5350
+Wire Notes Line
+	5550 6350 10300 6350
+Wire Notes Line
+	5550 2150 10300 2150
 $EndSCHEMATC

Commit message: daily updates
Parts:
- added J6: Conn_01x04, Connector_PinHeader_1.00mm:PinHeader_1x04_P1.00mm_Vertical_SMD_Pin1Left, symbol Connector_Generic:Conn_01x04
- U1: LCSC (none) -> C8304; LSCS C8304 -> (none)
Connections:
- net GND: now also J6.1 (Pin_1)
- net usb: now also J6.4 (Pin_4)
- net usb_dm: now also J6.3 (Pin_3)
- net usb_dp: now also J6.2 (Pin_2)
Changed lines of the file:
@@
 F 2 "Package_QFP:LQFP-48_7x7mm_P0.5mm" H 8150 3150 50  0001 R CNN
 F 3 "http://www.st.com/st-web-ui/static/active/en/resource/technical/document/datasheet/CD00161566.pdf" H 8750 4550 50  0001 C CNN
-F 4 "C8304" H 8750 4550 50  0001 C CNN "LSCS"
+F 4 "C8304" H 8750 4550 50  0001 C CNN "LCSC"
 	1    8750 4550
 	1    0    0    -1
@@
 Wire Notes Line
 	5550 2150 10300 2150
+$Comp
+L Connector_Generic:Conn_01x04 J6
+U 1 1 5F3ED892
+P 1450 4100
+F 0 "J6" H 1368 3675 50  0000 C CNN
+F 1 "Conn_01x04" H 1368 3766 50  0000 C CNN
+F 2 "Connector_PinHeader_1.00mm:PinHeader_1x04_P1.00mm_Vertical_SMD_Pin1Left" H 1450 4100 50  0001 C CNN
+F 3 "~" H 1450 4100 50  0001 C CNN
+	1    1450 4100
+	-1   0    0    1
+$EndComp
+Text Label 1650 3900 0    50   ~ 0
+usb
+$Comp
+L power:GND #PWR0115
+U 1 1 5F3EED8C
+P 1650 4200
+F 0 "#PWR0115" H 1650 3950 50  0001 C CNN
+F 1 "GND" H 1655 4027 50  0000 C CNN
+F 2 "" H 1650 4200 50  0001 C CNN
+F 3 "" H 1650 4200 50  0001 C CNN
+	1    1650 4200
+	1    0    0    -1
+$EndComp
+Text Label 1650 4100 0    50   ~ 0
+usb_dp
+Text Label 1650 4000 0    50   ~ 0
+usb_dm
 $EndSCHEMATC
